Commit message: Arm linked to torso and spinning on joint

File: dreadnought.urdf (robot description, URDF)
Before this commit: robot myfirst, 2 links, 1 joints
Links:
- removed link left_arm_link
- added link right_arm_link; visual mesh filename=file:///home/vivi/ws_moveit2/src/custom_robot/stl/Dreadnaug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 scale=0.1 0.1 0.1
- added link world
- link base_link: geometry visual mesh filename=file:///home/vivi/ws_moveit2/src/custom_robot/stl/Dreadnaug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 scale=0.1 0.1 0.1
Joints:
- removed joint base_to_right_arm
- added joint base_to_right_arm_joint: type continuous, parent base_link, child right_arm_link, origin xyz=0.8 1.7 2.2
- added joint world_to_base_joint: type fixed, parent world, child base_link, origin xyz=0 0 -0.5

Commit message: body with right and left arms

File: dreadnought.urdf (robot description, URDF)
Before this commit: robot dreadnought, 3 links, 2 joints
Links:
- added link left_arm_link; visual mesh filename=file:///home/vivi/ws_moveit2/src/custom_robot/stl/Dreadnaug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 scale=0.1 0.1 0.1
Joints:
- added joint base_to_left_arm_joint: type continuous, parent base_link, child left_arm_link, origin xyz=2.8 1.7 2.2

Commit message: readme for startup and minor tweaks to urdf

File: dreadnought.urdf (robot description, URDF)
Before this commit: robot dreadnought, 4 links, 3 joints
Links:
- added link legs_link; visual mesh filename=file:///home/vivi/ws_moveit2/src/custom_robot/stl/Dreadnoug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 scale=0.1 0.1 0.1
Joints:
- added joint base_to_legs_joint: type continuous, parent base_link, child legs_link, origin xyz=0.0 0 1.5
- joint world_to_base_joint: origin xyz=0 0 -0.5 -> xyz=1 1 0

Commit message: Legs in position under torso

File: dreadnought.urdf (robot description, URDF)
Before this commit: robot dreadnought, 5 links, 4 joints
Joints:
- joint base_to_legs_joint: axis (none) -> 0 0 1; origin xyz=0.0 0 1.5 -> xyz=1.75 1.75 1.5

Commit message: Spins on correct axis, issue with model being in wrong position on z axis

File: dreadnought.urdf (robot description, URDF)
Before this commit: robot dreadnought, 5 links, 4 joints
Links:
- removed link legs_link
- added link torso_link; visual mesh filename=file:///home/vivi/ws_moveit2/src/custom_robot/stl/Dreadnaug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 scale=0.1 0.1 0.1
- link base_link: geometry visual mesh filename=file:///home/vivi/ws_moveit2/src/custom_robot/stl/Dreadnoug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 scale=0.1 0.1 0.1
Joints:
- joint base_to_left_arm_joint: parent base_link -> torso_link
- joint base_to_legs_joint: child legs_link -> base_link; parent base_link -> torso_link
- joint base_to_right_arm_joint: parent base_link -> torso_link
- joint world_to_base_joint: child base_link -> torso_link

Commit message: Change arms to revolute joint types and rename torso to root link

File: dreadnought.urdf (robot description, URDF)
Before this commit: robot dreadnought, 5 links, 4 joints
Links:
- removed link torso_link
- added link root_link; visual mesh filename=file:///home/vivi/ws_moveit2/src/custom_robot/stl/Dreadnaug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 scale=0.1 0.1 0.1
Joints:
- removed joint base_to_left_arm_joint
- removed joint base_to_legs_joint
- removed joint base_to_right_arm_joint
- removed joint world_to_base_joint
- added joint torso_to_left_arm_joint: type revolute, parent root_link, child left_arm_link, origin xyz=2.8 1.7 2.2, limit lower=-2.5 upper=0.5 effort=1000.0 velocity=0.5
- added joint torso_to_legs_joint: type continuous, parent root_link, child base_link, origin xyz=1.75 1.75 1.5, axis 0 0 1
- added joint torso_to_right_arm_joint: type revolute, parent root_link, child right_arm_link, origin xyz=0.8 1.7 2.2, limit lower=-1.5 upper=0.5 effort=1000.0 velocity=0.5
- added joint world_to_torso_joint: type fixed, parent world, child root_link, origin xyz=1 1 0

Commit message: Bring the center of model out of zero on the z axis

File: dreadnought.urdf (robot description, URDF)
Before this commit: robot dreadnought, 5 links, 4 joints
Joints:
- joint torso_to_left_arm_joint: origin xyz=2.8 1.7 2.2 -> xyz=2.8 1.7 0.7
- joint torso_to_legs_joint: origin xyz=1.75 1.75 1.5 -> xyz=1.75 1.75 0
- joint torso_to_right_arm_joint: origin xyz=0.8 1.7 2.2 -> xyz=0.8 1.7 0.7

Commit message: Match link position to joints and switch torso and leg joint to revolute with around 90 degrees of movement (front facing)

File: dreadnought.urdf (robot description, URDF)
Before this commit: robot dreadnought, 5 links, 4 joints
Joints:
- joint torso_to_left_arm_joint: origin xyz=2.8 1.7 0.7 -> xyz=2.8 1.7 2.3
- joint torso_to_legs_joint: limit (none) -> lower=-1.5 upper=1.5 effort=1000.0 velocity=0.5; type continuous -> revolute
- joint torso_to_right_arm_joint: origin xyz=0.8 1.7 0.7 -> xyz=0.8 1.7 2.3
