Commit message: Make package for model

File: urdf/dreadnought.urdf (robot description, URDF)
Before this commit: robot dreadnought, 5 links, 4 joints
Links:
- link base_link: geometry visual mesh filename=package://dreadnought_urdf/stl/binary/DreadnoughtV1Legs-con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 scale=0.1 0.1 0.1
- link left_arm_link: geometry visual mesh filename=package://dreadnought_urdf/stl/binary/DreadnaughtV1larm-con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 scale=0.1 0.1 0.1
- link right_arm_link: geometry visual mesh filename=package://dreadnought_urdf/stl/binary/DreadnaughtV1RArm-con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 scale=0.1 0.1 0.1
- link root_link: geometry visual mesh filename=package://dreadnought_urdf/stl/binary/DreadnaughtV1Body-con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 scale=0.1 0.1 0.1
